Commit message: Scale model to torta size

File: tortasim_description/urdf/tortabot.gazebo.xacro (robot description, xacro)
@@ -1,4 +1,4 @@
 <?xml version="1.0"?>
-<robot name="hellobot_gazebo" xmlns:xacro="http://ros.org/wiki/xacro">
+<robot name="tortabot_gazebo" xmlns:xacro="http://ros.org/wiki/xacro">
     <gazebo reference="camera_link">
       <material>Gazebo/Green</material>
@@ -21,5 +21,5 @@
           <alwaysOn>true</alwaysOn>
           <updateRate>0.0</updateRate>
-          <cameraName>hellobot/camera</cameraName>
+          <cameraName>tortabot/camera</cameraName>
           <imageTopicName>image_raw</imageTopicName>
           <cameraInfoTopicName>camera_info</cameraInfoTopicName>
@@ -42,6 +42,6 @@
         <rightJoint>right_wheel_hinge</rightJoint>
         <wheelSeparation>0.30</wheelSeparation>
-        <wheelDiameter>0.2</wheelDiameter>
-        <torque>30</torque>
+        <wheelDiameter>0.08</wheelDiameter>
+        <torque>10</torque>
         <commandTopic>cmd_vel</commandTopic>
         <odometryTopic>odom</odometryTopic>
@@ -50,9 +50,9 @@
     </plugin>
     </gazebo>
-    <gazebo reference="chassis">
+    <!-- <gazebo reference="chassis">
         <material>
         Gazebo/Black
         </material>
-    </gazebo>
+    </gazebo>  -->
     <gazebo reference="left_wheel">
         <material>

File: tortasim_description/urdf/tortabot.xacro (robot description, xacro)
@@ -1,178 +1,178 @@
 <?xml version='1.0'?>
-<robot name="hellobot" xmlns:xacro="http://www.ros.org/wiki/xacro">
-    <xacro:include filename="$(find hellobot_specs)/urdf/materials.xacro"/>
-    <xacro:include filename="$(find hellobot_specs)/urdf/hellobot.gazebo.xacro"/>
-    <xacro:property name="cameraSize" value="0.05"/>
+<robot name="tortabot" xmlns:xacro="http://www.ros.org/wiki/xacro">
+    <xacro:include filename="$(find tortasim_description)/urdf/materials.xacro"/>
+    <xacro:include filename="$(find tortasim_description)/urdf/tortabot.gazebo.xacro"/>
+    <!-- <xacro:property name="cameraSize" value="0.01"/> -->
     <xacro:property name="cameraMass" value="0.1"/>
-      <link name="base_footprint" />
+    <link name="base_footprint" />
     <joint name="base_footprint_joint" type="fixed">
         <parent link="base_footprint" />
         <child link="chassis" />
     </joint>
-  <link name='chassis'>
-    <pose>0 0 0.1 0 0 0</pose>
-    <inertial>
-      <mass value="5.0"/>
-      <origin xyz="0.0 0 0.1" rpy=" 0 0 0"/>
-      <inertia
-          ixx="0.1" ixy="0" ixz="0"
-          iyy="0.1" iyz="0"
-          izz="0.1"
-      />
-    </inertial>
-    <collision name='collision'>
-      <geometry>
-        <box size=".4 .2 .1"/>
-      </geometry>
-    </collision>
-    <visual name='chassis_visual'>
-      <origin xyz="0 0 0" rpy=" 0 0 0"/>
-      <geometry>
-        <box size=".4 .2 .1"/>
-        <!-- <mesh filename="file://$(find hellobot_specs)/meshes/fixed_torta.dae" /> -->
-      </geometry>
-      <material name="black"/>
-    </visual>
-    <collision name='caster_collision'>
-      <origin xyz="-0.15 0 -0.05" rpy=" 0 0 0"/>
-      <geometry>
-        <sphere radius="0.05"/>
-      </geometry>
-      <!-- <surface>
-        <friction>
-          <ode>
-            <mu>0</mu>
-            <mu2>0</mu2>
-            <slip1>1.0</slip1>
-            <slip2>1.0</slip2>
-          </ode>
-        </friction>
-      </surface> -->
-    </collision>
-    <visual name='caster_visual'>
-      <origin xyz="-0.15 0 -0.05" rpy=" 0 0 0"/>
-      <geometry>
-        <sphere radius="0.05"/>
-      </geometry>
-      <material name="green">   </material>
-    </visual>
-    <collision name='caster_front_collision'>
-      <origin xyz="0.15 0 -0.05" rpy=" 0 0 0"/>
-      <geometry>
-        <sphere radius="0.05"/>
-      </geometry>
-      <!-- <surface>
-        <friction>
-          <ode>
-            <mu>0</mu>
-            <mu2>0</mu2>
-            <slip1>1.0</slip1>
-            <slip2>1.0</slip2>
-          </ode>
-        </friction>
-      </surface> -->
-    </collision>
-    <visual name='caster_front_visual'>
-      <origin xyz="0.15 0 -0.05" rpy=" 0 0 0"/>
-      <geometry>
-        <sphere radius="0.05"/>
-      </geometry>
-      <material name="green">   </material>
-    </visual>
-  </link>
-  <link name="left_wheel">
-    <!--origin xyz="0.1 0.13 0.1" rpy="0 1.5707 1.5707"/-->
-    <collision name="collision">
-      <origin xyz="0 0 0" rpy="0 1.5707 1.5707"/>
-      <geometry>
-        <cylinder radius="0.1" length="0.05"/>
-      </geometry>
-    </collision>
-    <visual name="left_wheel_visual">
-      <origin xyz="0 0 0" rpy="0 1.5707 1.5707"/>
-      <geometry>
-        <cylinder radius="0.1" length="0.05"/>
-      </geometry>
-      <material name="yellow"/>
-    </visual>
-    <inertial>
-      <origin xyz="0 0 0" rpy="0 1.5707 1.5707"/>
-      <mass value="5"/>
-      <inertia
-        ixx=".1" ixy="0.0" ixz="0.0"
-        iyy=".1" iyz="0.0"
-        izz=".1"/>
-    </inertial>
-  </link>
-  <link name="right_wheel">
-    <!--origin xyz="0.1 -0.13 0.1" rpy="0 1.5707 1.5707"/-->
-    <collision name="collision">
-      <origin xyz="0 0 0" rpy="0 1.5707 1.5707"/>
-      <geometry>
-        <cylinder radius="0.1" length="0.05"/>
-      </geometry>
-    </collision>
-    <visual name="right_wheel_visual">
-      <origin xyz="0 0 0" rpy="0 1.5707 1.5707"/>
-      <geometry>
-        <cylinder radius="0.1" length="0.05"/>
-      </geometry>
-      <material name="yellow"/>
-    </visual>
-    <inertial>
-      <origin xyz="0 0 0" rpy="0 1.5707 1.5707"/>
-      <mass value="5"/>
-      <inertia
-        ixx=".1" ixy="0.0" ixz="0.0"
-        iyy=".1" iyz="0.0"
-        izz=".1"/>
-    </inertial>
-  </link>
-  <joint type="continuous" name="left_wheel_hinge">
-    <origin xyz="0 0.15 0" rpy="0 0 0"/>
-    <!--origin xyz="0.1 0.13 0" rpy="0 1.5707 1.5707"/-->
-    <child link="left_wheel"/>
-    <parent link="chassis"/>
-    <axis xyz="0 1 0" rpy="0 0 0"/>
-    <!-- <limit effort="10000" velocity="1000"/> -->
-    <joint_properties damping="0.0" friction="0.0"/>
-  </joint>
-  <joint type="continuous" name="right_wheel_hinge">
-    <origin xyz="0 -0.15 0" rpy="0 0 0"/>
-    <!--origin xyz="0.1 -0.13 0" rpy="0 1.5707 1.5707"/-->
-    <child link="right_wheel"/>
-    <parent link="chassis"/>
-    <axis xyz="0 1 0" rpy="0 0 0"/>
-    <!-- <limit effort="10000" velocity="1000"/> -->
-    <joint_properties damping="0.0" friction="0.0"/>
-  </joint>
-  <!-- Camera -->
-  <link name="camera_link">
-    <collision>
-      <origin xyz="0 0 0" rpy="0 0 0"/>
-      <geometry>
-        <box size="${cameraSize} ${cameraSize} ${cameraSize}"/>
-      </geometry>
-    </collision>
-    <visual>
-      <origin xyz="0 0 0" rpy="0 0 0"/>
-      <geometry>
-        <box size="${cameraSize} ${cameraSize} ${cameraSize}"/>
-      </geometry>
-      <material name="green"/>
-    </visual>
-    <inertial>
-      <mass value="${cameraMass}" />
-      <origin xyz="0 0 0" rpy="0 0 0"/>
-      <box_inertia m="${cameraMass}" x="${cameraSize}" y="${cameraSize}" z="${cameraSize}" />
-      <inertia ixx="1e-6" ixy="0" ixz="0" iyy="1e-6" iyz="0" izz="1e-6" />
-    </inertial>
-  </link>
-  <joint name="camera_joint" type="fixed">
-    <axis xyz="0 1 0" />
-    <origin xyz=".2 0 0" rpy="0 0 0"/>
-    <parent link="chassis"/>
-    <child link="camera_link"/>
-  </joint>
+    <link name='chassis'>
+      <pose>0 0 0.1 0 0 0</pose>
+      <inertial>
+        <mass value="5.0"/>
+        <origin xyz="0.0 0 0.1" rpy=" 0 0 0"/>
+        <inertia
+            ixx="0.1" ixy="0" ixz="0"
+            iyy="0.1" iyz="0"
+            izz="0.1"
+        />
+      </inertial>
+      <collision name='collision'>
+        <geometry>
+          <box size=".3 .3 .1"/>
+        </geometry>
+      </collision>
+      <visual name='chassis_visual'>
+        <origin xyz="0 0 -0.05" rpy=" 0 0 1.57"/>
+        <geometry>
+          <!-- <box size=".3 .3 .1"/> -->
+          <mesh filename="file://$(find tortasim_description)/meshes/torta_v1_1.dae" />
+        </geometry>
+        <!-- <material name="black"/> -->
+      </visual>
+      <collision name='caster_collision'>
+        <origin xyz="-0.15 0 -0.025" rpy=" 0 0 0"/>
+        <geometry>
+          <sphere radius="0.025"/>
+        </geometry>
+        <!-- <surface>
+          <friction>
+            <ode>
+              <mu>0</mu>
+              <mu2>0</mu2>
+              <slip1>1.0</slip1>
+              <slip2>1.0</slip2>
+            </ode>
+          </friction>
+        </surface> -->
+      </collision>
+      <visual name='caster_visual'>
+        <origin xyz="-0.15 0 -0.025" rpy=" 0 0 0"/>
+        <geometry>
+          <sphere radius="0.025"/>
+        </geometry>
+        <material name="green">   </material>
+      </visual>
+      <collision name='caster_front_collision'>
+        <origin xyz="0.15 0 -0.025" rpy=" 0 0 0"/>
+        <geometry>
+          <sphere radius="0.025"/>
+        </geometry>
+        <!-- <surface>
+          <friction>
+            <ode>
+              <mu>0</mu>
+              <mu2>0</mu2>
+              <slip1>1.0</slip1>
+              <slip2>1.0</slip2>
+            </ode>
+          </friction>
+        </surface> -->
+      </collision>
+      <visual name='caster_front_visual'>
+        <origin xyz="0.15 0 -0.025" rpy=" 0 0 0"/>
+        <geometry>
+          <sphere radius="0.025"/>
+        </geometry>
+        <material name="green">   </material>
+      </visual>
+    </link>
+    <link name="left_wheel">
+      <!--origin xyz="0.1 0.13 0.1" rpy="0 1.5707 1.5707"/-->
+      <collision name="collision">
+        <origin xyz="0 0 0" rpy="0 1.5707 1.5707"/>
+        <geometry>
+          <cylinder radius="0.05" length="0.02"/>
+        </geometry>
+      </collision>
+      <visual name="left_wheel_visual">
+        <origin xyz="0 0 0" rpy="0 1.5707 1.5707"/>
+        <geometry>
+          <cylinder radius="0.05" length="0.02"/>
+        </geometry>
+        <material name="yellow"/>
+      </visual>
+      <inertial>
+        <origin xyz="0 0 0" rpy="0 1.5707 1.5707"/>
+        <mass value="5"/>
+        <inertia
+          ixx=".1" ixy="0.0" ixz="0.0"
+          iyy=".1" iyz="0.0"
+          izz=".1"/>
+      </inertial>
+    </link>
+    <link name="right_wheel">
+      <!--origin xyz="0.1 -0.13 0.1" rpy="0 1.5707 1.5707"/-->
+      <collision name="collision">
+        <origin xyz="0 0 0" rpy="0 1.5707 1.5707"/>
+        <geometry>
+          <cylinder radius="0.05" length="0.02"/>
+        </geometry>
+      </collision>
+      <visual name="right_wheel_visual">
+        <origin xyz="0 0 0" rpy="0 1.5707 1.5707"/>
+        <geometry>
+          <cylinder radius="0.05" length="0.02"/>
+        </geometry>
+        <material name="yellow"/>
+      </visual>
+      <inertial>
+        <origin xyz="0 0 0" rpy="0 1.5707 1.5707"/>
+        <mass value="5"/>
+        <inertia
+          ixx=".1" ixy="0.0" ixz="0.0"
+          iyy=".1" iyz="0.0"
+          izz=".1"/>
+      </inertial>
+    </link>
+    <joint type="continuous" name="left_wheel_hinge">
+      <origin xyz="0 0.17 0" rpy="0 0 0"/>
+      <!--origin xyz="0.1 0.13 0" rpy="0 1.5707 1.5707"/-->
+      <child link="left_wheel"/>
+      <parent link="chassis"/>
+      <axis xyz="0 1 0" rpy="0 0 0"/>
+      <!-- <limit effort="10000" velocity="1000"/> -->
+      <joint_properties damping="0.0" friction="0.0"/>
+    </joint>
+    <joint type="continuous" name="right_wheel_hinge">
+      <origin xyz="0 -0.17 0" rpy="0 0 0"/>
+      <!--origin xyz="0.1 -0.13 0" rpy="0 1.5707 1.5707"/-->
+      <child link="right_wheel"/>
+      <parent link="chassis"/>
+      <axis xyz="0 1 0" rpy="0 0 0"/>
+      <!-- <limit effort="10000" velocity="1000"/> -->
+      <joint_properties damping="0.0" friction="0.0"/>
+    </joint>
+    <!-- Camera -->
+    <link name="camera_link">
+      <collision>
+        <origin xyz="0 0 0" rpy="0 0 0"/>
+        <geometry>
+          <box size="0.005 0.05 0.015"/>
+        </geometry>
+      </collision>
+      <visual>
+        <origin xyz="0 0 0" rpy="0 0 0"/>
+        <geometry>
+          <box size="0.005 0.05 0.015"/>
+        </geometry>
+        <material name="green"/>
+      </visual>
+      <inertial>
+        <mass value="${cameraMass}" />
+        <origin xyz="0 0 0" rpy="0 0 0"/>
+        <box_inertia m="${cameraMass}" x="0.005" y="0.05" z="0.015" />
+        <inertia ixx="1e-6" ixy="0" ixz="0" iyy="1e-6" iyz="0" izz="1e-6" />
+      </inertial>
+    </link>
+    <joint name="camera_joint" type="fixed">
+      <axis xyz="0 1 0" />
+      <origin xyz=".09 0 0.16" rpy="0 0 0"/>
+      <parent link="chassis"/>
+      <child link="camera_link"/>
+    </joint>
   <!-- Hokuyo Laser
   <link name="hokuyo_link">

Commit message: Include IMU and StereoCamera

File: tortasim_description/urdf/tortabot.gazebo.xacro (robot description, xacro)
@@ -1,4 +1,91 @@
 <?xml version="1.0"?>
 <robot name="tortabot_gazebo" xmlns:xacro="http://ros.org/wiki/xacro">
+  <gazebo>
+    <plugin name="imu_plugin" filename="libgazebo_ros_imu.so">
+      <alwaysOn>true</alwaysOn>
+      <bodyName>chassis</bodyName>
+      <topicName>imu</topicName>
+      <serviceName>imu_service</serviceName>
+      <gaussianNoise>1.0</gaussianNoise>
+      <updateRate>20.0</updateRate>
+    </plugin>
+  </gazebo>
+  <gazebo reference="imu_link">
+    <material>Gazebo/Blue</material>
+    <gravity>true</gravity>
+    <sensor name="imu_sensor" type="imu">
+      <always_on>true</always_on>
+      <update_rate>100</update_rate>
+      <visualize>true</visualize>
+      <topic>__default_topic__</topic>
+      <plugin filename="libgazebo_ros_imu_sensor.so" name="imu_plugin">
+        <topicName>imu</topicName>
+        <bodyName>imu_link</bodyName>
+        <updateRateHZ>20.0</updateRateHZ>
+        <gaussianNoise>0.0</gaussianNoise>
+        <xyzOffset>0 0 0</xyzOffset>
+        <rpyOffset>0 0 0</rpyOffset>
+        <frameName>imu_link</frameName>
+        <initialOrientationAsReference>false</initialOrientationAsReference>
+      </plugin>
+      <pose>0 0 0 0 0 0</pose>
+    </sensor>
+  </gazebo>
+  <gazebo reference="stereo_camera_link">
+    <material>Gazebo/Green</material>
+    <sensor type="multicamera" name="stereo_camera">
+      <update_rate>30.0</update_rate>
+      <camera name="left">
+        <horizontal_fov>1.3962634</horizontal_fov>
+        <image>
+          <width>800</width>
+          <height>800</height>
+          <format>R8G8B8</format>
+        </image>
+        <clip>
+          <near>0.02</near>
+          <far>300</far>
+        </clip>
+        <noise>
+          <type>gaussian</type>
+          <mean>0.0</mean>
+          <stddev>0.007</stddev>
+        </noise>
+      </camera>
+      <camera name="right">
+        <pose>0 -0.07 0 0 0 0</pose>
+        <horizontal_fov>1.3962634</horizontal_fov>
+        <image>
+          <width>800</width>
+          <height>800</height>
+          <format>R8G8B8</format>
+        </image>
+        <clip>
+          <near>0.02</near>
+          <far>300</far>
+        </clip>
+        <noise>
+          <type>gaussian</type>
+          <mean>0.0</mean>
+          <stddev>0.007</stddev>
+        </noise>
+      </camera>
+      <plugin name="stereo_camera_controller" filename="libgazebo_ros_multicamera.so">
+        <alwaysOn>true</alwaysOn>
+        <updateRate>0.0</updateRate>
+        <cameraName>tortabot/camera</cameraName>
+        <imageTopicName>image_raw</imageTopicName>
+        <cameraInfoTopicName>camera_info</cameraInfoTopicName>
+        <frameName>left_camera_optical_frame</frameName>
+        <!--<rightFrameName>right_camera_optical_frame</rightFrameName>-->
+        <hackBaseline>0.07</hackBaseline>
+        <distortionK1>0.0</distortionK1>
+        <distortionK2>0.0</distortionK2>
+        <distortionK3>0.0</distortionK3>
+        <distortionT1>0.0</distortionT1>
+        <distortionT2>0.0</distortionT2>
+      </plugin>
+    </sensor>
+  </gazebo>
     <gazebo reference="camera_link">
       <material>Gazebo/Green</material>
@@ -65,35 +152,3 @@
         </material>
     </gazebo>
-    <!-- hokuyo -->
-  <!-- <gazebo reference="hokuyo_link">
-    <sensor type="gpu_ray" name="head_hokuyo_sensor">
-      <pose>0 0 0 0 0 0</pose>
-      <visualize>ture</visualize>
-      <update_rate>40</update_rate>
-      <ray>
-        <scan>
-          <horizontal>
-            <samples>720</samples>
-            <resolution>1</resolution>
-            <min_angle>-1.570796</min_angle>
-            <max_angle>1.570796</max_angle>
-          </horizontal>
-        </scan>
-        <range>
-          <min>0.10</min>
-          <max>30.0</max>
-          <resolution>0.01</resolution>
-        </range>
-        <noise>
-          <type>gaussian</type>
-          <mean>0.0</mean>
-          <stddev>0.01</stddev>
-        </noise>
-      </ray>
-      <plugin name="gazebo_ros_head_hokuyo_controller" filename="libgazebo_ros_gpu_laser.so">
-        <topicName>/hellobot/laser/scan</topicName>
-        <frameName>hokuyo_link</frameName>
-      </plugin>
-    </sensor>
-  </gazebo> -->
 </robot>

File: tortasim_description/urdf/tortabot.xacro (robot description, xacro)
@@ -148,5 +148,5 @@
     </joint>
     <!-- Camera -->
-    <link name="camera_link">
+    <link name="stereo_camera_link">
       <collision>
         <origin xyz="0 0 0" rpy="0 0 0"/>
@@ -173,5 +173,32 @@
       <origin xyz=".09 0 0.16" rpy="0 0 0"/>
       <parent link="chassis"/>
-      <child link="camera_link"/>
+      <child link="stereo_camera_link"/>
+    </joint>
+    <!-- IMU -->
+    <link name="imu_link">
+      <collision>
+        <origin xyz="0 0 0" rpy="0 0 0"/>
+        <geometry>
+          <box size="0.02 0.02 0.005"/>
+        </geometry>
+      </collision>
+      <visual>
+        <origin xyz="0 0 0" rpy="0 0 0"/>
+        <geometry>
+          <box size="0.02 0.02 0.005"/>
+        </geometry>
+        <material name="Blue"/>
+      </visual>
+      <inertial>
+        <mass value="0.05" />
+        <origin xyz="0 0 0" rpy="0 0 0"/>
+        <box_inertia m="0.05" x="0.005" y="0.05" z="0.015" />
+        <inertia ixx="1e-6" ixy="0" ixz="0" iyy="1e-6" iyz="0" izz="1e-6" />
+      </inertial>
+    </link>
+    <joint name="IMU_joint" type="fixed">
+      <origin xyz="0 0 0.06" rpy="0 0 0"/>
+      <parent link="chassis"/>
+      <child link="imu_link"/>
     </joint>
   <!-- Hokuyo Laser

Commit message: Add Lidar A1 Model

File: tortasim_description/urdf/tortabot.gazebo.xacro (robot description, xacro)
@@ -1,4 +1,6 @@
 <?xml version="1.0"?>
 <robot name="tortabot_gazebo" xmlns:xacro="http://ros.org/wiki/xacro">
+  <xacro:arg name="laser_visual" default="false"/>
+  <xacro:arg name="imu_visual"   default="false"/>
   <gazebo>
     <plugin name="imu_plugin" filename="libgazebo_ros_imu.so">
@@ -137,4 +139,36 @@
     </plugin>
     </gazebo>
+    <gazebo reference="base_scan">
+      <material>Gazebo/FlatBlack</material>
+      <sensor type="ray" name="lds_lfcd_sensor">
+        <pose>0 0 0 0 0 0</pose>
+        <visualize>$(arg laser_visual)</visualize>
+        <update_rate>5</update_rate>
+        <ray>
+          <scan>
+            <horizontal>
+              <samples>360</samples>
+              <resolution>1</resolution>
+              <min_angle>0.0</min_angle>
+              <max_angle>6.28319</max_angle>
+            </horizontal>
+          </scan>
+          <range>
+            <min>0.120</min>
+            <max>3.5</max>
+            <resolution>0.015</resolution>
+          </range>
+          <noise>
+            <type>gaussian</type>
+            <mean>0.0</mean>
+            <stddev>0.01</stddev>
+          </noise>
+        </ray>
+        <plugin name="gazebo_ros_lds_lfcd_controller" filename="libgazebo_ros_laser.so">
+          <topicName>scan</topicName>
+          <frameName>base_scan</frameName>
+        </plugin>
+      </sensor>
+    </gazebo>
     <!-- <gazebo reference="chassis">
         <material>

File: tortasim_description/urdf/tortabot.xacro (robot description, xacro)
@@ -195,4 +195,31 @@
         <box_inertia m="0.05" x="0.005" y="0.05" z="0.015" />
         <inertia ixx="1e-6" ixy="0" ixz="0" iyy="1e-6" iyz="0" izz="1e-6" />
+      </inertial>
+    </link>
+    <joint name="scan_joint" type="fixed">
+      <parent link="chassis"/>
+      <child link="base_scan"/>
+      <origin xyz="-0.032 0 0.172" rpy="0 0 0"/>
+    </joint>
+    <link name="base_scan">
+      <visual>
+        <origin xyz="0 0 0.0" rpy="0 0 0"/>
+        <geometry>
+          <cylinder length="0.0315" radius="0.055"/>
+        </geometry>
+        <material name="red"/>
+      </visual>
+      <collision>
+        <origin xyz="0.015 0 -0.0065" rpy="0 0 0"/>
+        <geometry>
+          <cylinder length="0.0315" radius="0.055"/>
+        </geometry>
+      </collision>
+      <inertial>
+        <mass value="0.114" />
+        <origin xyz="0 0 0" />
+        <inertia ixx="0.001" ixy="0.0" ixz="0.0"
+                 iyy="0.001" iyz="0.0"
+                 izz="0.001" />
       </inertial>
     </link>
